Commit message: docker ros_robot update

File: kwj_description/urdf/kwj.urdf.xacro (robot description, xacro)
@@ -60,5 +60,5 @@
     <parent link="base_link"/>
     <child link="wheel_left_link"/>
-    <origin xyz="-0.0655 0.075 -0.02" rpy="-1.57 0 0"/>
+    <origin xyz="-0.0355 0.075 -0.02" rpy="-1.57 0 0"/>
     <axis xyz="0 0 1"/>
    </joint>
@@ -88,5 +88,5 @@
     <parent link="base_link"/>
     <child link="wheel_right_link"/>
-    <origin xyz="-0.0655 -0.0775 -0.02" rpy="-1.57 0 0"/>
+    <origin xyz="-0.0355 -0.0775 -0.02" rpy="-1.57 0 0"/>
     <axis xyz="0 0 1"/>
    </joint>

Commit message: foxy update

File: kwj_description/urdf/kwj.urdf.xacro (robot description, xacro)
@@ -57,9 +57,10 @@
     </inertial>
   </link>
-   <joint name="wheel_left_joint" type="fixed">
+   <joint name="wheel_left_joint" type="revolute">
     <parent link="base_link"/>
     <child link="wheel_left_link"/>
     <origin xyz="-0.0355 0.075 -0.02" rpy="-1.57 0 0"/>
     <axis xyz="0 0 1"/>
+    <limit lower="-3.14" upper="3.14" effort="30" velocity="10"/>
    </joint>
    <link name="wheel_left_link">
@@ -85,9 +86,10 @@
       </inertial>
   </link>
-   <joint name="wheel_right_joint" type="fixed">
+   <joint name="wheel_right_joint" type="revolute">
     <parent link="base_link"/>
     <child link="wheel_right_link"/>
     <origin xyz="-0.0355 -0.0775 -0.02" rpy="-1.57 0 0"/>
     <axis xyz="0 0 1"/>
+    <limit lower="-3.14" upper="3.14" effort="30" velocity="10"/>
    </joint>
    <link name="wheel_right_link">
