Commit message: foxy.launch.py launch success, and navigation2 success

File: kwj_description/urdf/kwj.gazebo.xacro (robot description, xacro)
@@ -2,73 +2,27 @@
 <robot name="KWJBot" xmlns:xacro="http://ros.org/wiki/xacro">
   <link name="base_footprint"/>
- <joint name="base_joint" type="fixed">
-  <parent link="base_footprint"/>
-  <child link="base_link"/>
-   <origin xyz="0 0 0.065" rpy="0 0 0"/>
- </joint>
+    <joint name="base_joint" type="fixed">
+       <parent link="base_footprint"/>
+       <child link="base_link"/>
+       <origin xyz="0 0 0.065" rpy="0 0 0"/>
+    </joint>
   <link name="base_link">
-    <visual>
-      <geometry>
-        <box size="0.5 0.5 0.2"/>
-      </geometry>
-      <material name="blue">
-        <color rgba="0 0 1 1"/>
-      </material>
-    </visual>
-    <collision>
-      <geometry>
-        <box size="0.5 0.5 0.2"/>
-      </geometry>
-    </collision>
-    <inertial>
-      <mass value="10.0"/>
-      <origin rpy="0 0 0" xyz="0 0 0"/>
-      <inertia ixx="0.1" ixy="0.0" ixz="0.0" iyy="0.1" iyz="0.0" izz="0.1"/>
-    </inertial>
-  </link>
-  <link name="wheel_left_link">
-    <visual>
-      <geometry>
-        <cylinder length="0.05" radius="0.1"/>
-      </geometry>
-      <material name="black">
-        <color rgba="0 0 0 1"/>
-      </material>
-    </visual>
-    <collision>
-      <geometry>
-        <cylinder length="0.05" radius="0.1"/>
-      </geometry>
-    </collision>
-    <inertial>
-      <mass value="1.0"/>
-      <origin rpy="0 0 0" xyz="0 0 0"/>
-      <inertia ixx="0.01" ixy="0.0" ixz="0.0" iyy="0.01" iyz="0.0" izz="0.01"/>
-    </inertial>
-  </link>
-  <link name="wheel_right_link">
-    <visual>
-      <geometry>
-        <cylinder length="0.05" radius="0.1"/>
-      </geometry>
-      <material name="black">
-        <color rgba="0 0 0 1"/>
-      </material>
-    </visual>
-    <collision>
-      <geometry>
-        <cylinder length="0.05" radius="0.1"/>
-      </geometry>
-    </collision>
-    <inertial>
-      <mass value="1.0"/>
-      <origin rpy="0 0 0" xyz="0 0 0"/>
-      <inertia ixx="0.01" ixy="0.0" ixz="0.0" iyy="0.01" iyz="0.0" izz="0.01"/>
-    </inertial>
-  </link>
-  <link name="caster_front_link">
-    <visual>
-      <geometry>
-        <sphere radius="0.05"/>
+    <inertial>
+      <origin xyz="0 0 0" rpy="0 0 0"/>
+      <mass value="1.0" />
+      <inertia ixx="0.001" ixy="0" ixz="0"
+               iyy="0.001" iyz="0"
+               izz="0.001" />
+      </inertial>
+    <collision>
+      <origin xyz="0 0 0" rpy="0 0 0"/>
+      <geometry>
+        <box size="0.155 0.2 0.25"/>
+      </geometry>
+    </collision>
+    <visual>
+      <origin xyz="0 0 0" rpy="0 0 0"/>
+      <geometry>
+        <mesh filename="package://kwj_description/meshes/base_link.stl" scale="1.0 1.0 1.0"/>
       </geometry>
       <material name="grey">
@@ -76,110 +30,140 @@
       </material>
     </visual>
-    <collision>
-      <geometry>
-        <sphere radius="0.05"/>
-      </geometry>
-    </collision>
-    <inertial>
-      <mass value="0.5"/>
-      <origin rpy="0 0 0" xyz="0 0 0"/>
-      <inertia ixx="0.005" ixy="0.0" ixz="0.0" iyy="0.005" iyz="0.0" izz="0.005"/>
+  </link>
+   <joint name="wheel_left_joint" type="fixed">
+    <parent link="base_link"/>
+    <child link="wheel_left_link"/>
+    <origin xyz="-0.0355 0.075 -0.02" rpy="-1.57 0 0"/>
+    <axis xyz="0 0 1"/>
+   </joint>
+   <link name="wheel_left_link">
+    <visual>
+      <origin xyz="0 0 0" rpy="0 0 0"/>
+        <geometry>
+         <cylinder length="0.026" radius="0.0335"/>
+        </geometry>
+      <material name="dark"/>
+    </visual>
+    <collision>
+      <origin xyz="0 0 0" rpy="0 0 0"/>
+      <geometry>
+        <cylinder length="0.026" radius="0.0335"/>
+      </geometry>
+    </collision>
+    <inertial>
+      <origin xyz="0 0 0" />
+      <mass value="2.8498940e-02" />
+      <inertia ixx="0.001" ixy="0" ixz="0"
+               iyy="0.001" iyz="0"
+               izz="0.001" />
+      </inertial>
+  </link>
+   <joint name="wheel_right_joint" type="fixed">
+    <parent link="base_link"/>
+    <child link="wheel_right_link"/>
+    <origin xyz="-0.0355 -0.0775 -0.02" rpy="-1.57 0 0"/>
+    <axis xyz="0 0 1"/>
+   </joint>
+   <link name="wheel_right_link">
+    <visual>
+      <origin xyz="0 0 0" rpy="0 0 0"/>
+       <geometry>
+         <cylinder length="0.026" radius="0.0335"/>
+       </geometry>
+      <material name="dark"/>
+    </visual>
+    <collision>
+      <origin xyz="0 0 0" rpy="0 0 0"/>
+      <geometry>
+        <cylinder length="0.026" radius="0.0335"/>
+      </geometry>
+    </collision>
+    <inertial>
+      <origin xyz="0 0 0" />
+      <mass value="2.8498940e-02" />
+      <inertia ixx="0.001" ixy="0" ixz="0"
+               iyy="0.001" iyz="0"
+               izz="0.001" />
+      </inertial>
+  </link>
+  <joint name="camera_joint" type="fixed">
+    <parent link="base_link"/>
+    <child link="camera_link"/>
+    <origin xyz="0.08 0 0.13" rpy="0 0 0"/>
+  </joint>
+  <link name="camera_link">
+    <visual>
+      <origin xyz="0 0 0" rpy="0 0 0"/>
+      <geometry>
+        <box size="0.03 0.07 0.03"/>
+      </geometry>
+      <material name="black"/>
+    </visual>
+    <collision>
+      <origin xyz="0 0 0" rpy="0 0 0"/>
+      <geometry>
+        <box size="0.1 0.1 0.05"/>
+      </geometry>
+    </collision>
+    <inertial>
+      <mass value="0.1"/>
+      <origin xyz="0 0 0" rpy="0 0 0"/>
+      <inertia ixx="0.01" iyy="0.01" izz="0.01" ixy="0" ixz="0" iyz="0"/>
     </inertial>
   </link>
-  <link name="imu_link">
-    <visual>
-      <geometry>
-        <box size="0.1 0.1 0.05"/>
-      </geometry>
-      <material name="grey">
-        <color rgba="0 0 0 1"/>
-      </material>
-    </visual>
-    <collision>
-      <geometry>
-        <box size="0.1 0.1 0.05"/>
-      </geometry>
-    </collision>
-    <inertial>
-      <mass value="0.2"/>
-      <origin rpy="0 0 0" xyz="0 0 0"/>
-      <inertia ixx="0.001" ixy="0.0" ixz="0.0" iyy="0.001" iyz="0.0" izz="0.001"/>
+  <joint name="caster_front_joint" type="fixed">
+    <parent link="base_link"/>
+    <child link="caster_front_link"/>
+    <origin xyz="0.193 0.01 -0.02" rpy="0 0 -1.57"/>
+  </joint>
+  <link name="caster_front_link">
+    <collision>
+      <origin xyz="0 0 0" rpy="0 0 0"/>
+      <geometry>
+        <cylinder length="0.016" radius="0.0175"/>
+      </geometry>
+    </collision>
+    <inertial>
+      <origin xyz="0 0 0" />
+      <mass value="0.005" />
+      <inertia ixx="0.001" ixy="0.0" ixz="0.0"
+               iyy="0.001" iyz="0.0"
+               izz="0.001" />
     </inertial>
   </link>
-  <link name="laser_link">
-    <visual>
-      <geometry>
-        <cylinder length="0.02" radius="0.05"/>
-      </geometry>
-      <material name="black">
-        <color rgba="0 0 0 1"/>
-      </material>
-    </visual>
-    <collision>
-      <geometry>
-        <cylinder length="0.02" radius="0.05"/>
-      </geometry>
-    </collision>
-    <inertial>
-      <mass value="0.1"/>
-      <origin rpy="0 0 0" xyz="0 0 0"/>
-      <inertia ixx="0.0001" ixy="0.0" ixz="0.0" iyy="0.0001" iyz="0.0" izz="0.0001"/>
+   <joint name="imu_joint" type="fixed">
+    <parent link="base_link"/>
+    <child link="imu_link"/>
+    <origin xyz="-0.07 0 0" rpy="0 0 0"/>
+   </joint>
+   <link name="imu_link"/>
+   <joint name="scan_joint" type="fixed">
+    <parent link="base_link"/>
+    <child link="laser_link"/>
+    <origin xyz="0.11 0 0.18" rpy="0 0 0"/>
+   </joint>
+   <link name="laser_link">
+    <visual>
+      <origin xyz="0 0 0" rpy="0 0 0"/>
+        <geometry>
+         <cylinder length="0.0105" radius="0.03435"/>
+      </geometry>
+      <material name="dark"/>
+    </visual>
+    <collision>
+      <origin xyz="0.055 0 0.2" rpy="0 0 0"/>
+      <geometry>
+        <cylinder length="0.0105" radius="0.03435"/>
+      </geometry>
+    </collision>
+    <inertial>
+      <mass value="0.114" />
+      <origin xyz="0 0 0" />
+      <inertia ixx="0.001" ixy="0.0" ixz="0.0"
+               iyy="0.001" iyz="0.0"
+               izz="0.001" />
     </inertial>
   </link>
-  <link name="camera_link">
-    <visual>
-      <geometry>
-        <box size="0.1 0.1 0.05"/>
-      </geometry>
-      <material name="black">
-        <color rgba="0 0 0 1"/>
-      </material>
-    </visual>
-    <collision>
-      <geometry>
-        <box size="0.1 0.1 0.05"/>
-      </geometry>
-    </collision>
-    <inertial>
-      <mass value="0.3"/>
-      <origin rpy="0 0 0" xyz="0 0 0"/>
-      <inertia ixx="0.002" ixy="0.0" ixz="0.0" iyy="0.002" iyz="0.0" izz="0.002"/>
-    </inertial>
-  </link>
-  <joint name="wheel_left_joint" type="revolute">
-    <parent link="base_link"/>
-    <child link="wheel_left_link"/>
-    <origin rpy="0 0 0" xyz="0.2 0.15 0"/>
-    <axis xyz="0 1 0"/>
-    <limit effort="10" lower="-1.57" upper="1.57" velocity="1"/>
-  </joint>
-  <joint name="wheel_right_joint" type="revolute">
-    <parent link="base_link"/>
-    <child link="wheel_right_link"/>
-    <origin rpy="0 0 0" xyz="0.2 -0.15 0"/>
-    <axis xyz="0 1 0"/>
-    <limit effort="10" lower="-1.57" upper="1.57" velocity="1"/>
-  </joint>
-  <joint name="caster_front_joint" type="fixed">
-    <parent link="base_link"/>
-    <child link="caster_front_link"/>
-    <origin rpy="0 0 0" xyz="0 -0.2 0"/>
-  </joint>
-  <joint name="imu_joint" type="fixed">
-    <parent link="base_link"/>
-    <child link="imu_link"/>
-    <origin rpy="0 0 0" xyz="0 0 0.1"/>
-  </joint>
-  <joint name="laser_joint" type="fixed">
-    <parent link="base_link"/>
-    <child link="laser_link"/>
-    <origin rpy="0 0 0" xyz="0.3 0 0.1"/>
-  </joint>
-  <joint name="camera_joint" type="fixed">
-    <parent link="base_link"/>
-    <child link="camera_link"/>
-    <origin rpy="0 0 0" xyz="-0.3 0 0.1"/>
-  </joint>
-  <!-- Gazebo 설정 추가 -->
+  <!-- Gazebo -->
   <gazebo reference="base_link">
     <material>Gazebo/DarkGrey</material>
@@ -233,9 +217,4 @@
       </noise>
     </imu>
-    <plugin name="imu_plugin" filename="libgazebo_ros_imu_sensor.so">
-      <remapping>~/imu_plugin/out:=imu/data</remapping>
-      <bodyName>imu_link</bodyName>
-      <updateRate>10</updateRate>
-    </plugin>
     <plugin name="imu_plugin" filename="libgazebo_ros_imu_sensor.so">
           <ros>

File: kwj_description/urdf/kwjbot.urdf (robot description, URDF)
Before this commit: robot KWJBot, 8 links, 7 joints
Links:
- link base_link: mass 10.0 -> 1.0; geometry collision box size=0.155 0.2 0.25; visual mesh filename=package://kwj_description/meshes/base_link.stl scale=1.0 1.0 1.0
- link camera_link: mass 0.3 -> 0.1; geometry collision box size=0.1 0.1 0.05; visual box size=0.03 0.07 0.03
- link caster_front_link: mass 0.5 -> 0.005; geometry collision cylinder length=0.016 radius=0.0175
- link imu_link: mass 0.2 -> None; geometry 
- link laser_link: mass 0.1 -> 0.114; geometry collision cylinder length=0.0105 radius=0.03435; visual cylinder length=0.0105 radius=0.03435
- link wheel_left_link: mass 1.0 -> 2.8498940e-02; geometry collision cylinder length=0.026 radius=0.0335; visual cylinder length=0.026 radius=0.0335
- link wheel_right_link: mass 1.0 -> 2.8498940e-02; geometry collision cylinder length=0.026 radius=0.0335; visual cylinder length=0.026 radius=0.0335
Joints:
- removed joint laser_joint
- added joint scan_joint: type fixed, parent base_link, child laser_link, origin xyz=0.11 0 0.18 rpy=0 0 0
- joint camera_joint: origin xyz=-0.3 0 0.1 rpy=0 0 0 -> xyz=0.08 0 0.13 rpy=0 0 0
- joint caster_front_joint: origin xyz=0 -0.2 0 rpy=0 0 0 -> xyz=0.193 0.01 -0.02 rpy=0 0 -1.57
- joint imu_joint: origin xyz=0 0 0.1 rpy=0 0 0 -> xyz=-0.07 0 0 rpy=0 0 0
- joint wheel_left_joint: axis 0 1 0 -> 0 0 1; limit lower=-1.57 upper=1.57 effort=10 velocity=1 -> (none); origin xyz=0.2 0.15 0 rpy=0 0 0 -> xyz=-0.0355 0.075 -0.02 rpy=-1.57 0 0; type revolute -> fixed
- joint wheel_right_joint: axis 0 1 0 -> 0 0 1; limit lower=-1.57 upper=1.57 effort=10 velocity=1 -> (none); origin xyz=0.2 -0.15 0 rpy=0 0 0 -> xyz=-0.0355 -0.0775 -0.02 rpy=-1.57 0 0; type revolute -> fixed
